File: PathFinder KiCad/PathFinder KiCad.kicad_pcb (KiCad board)
At the start: 2 copper layers, 41.5 x 59 mm, 12 parts, among them J1 Conn_01x02_Socket, SW1 SW_Push, SW2 SW_Push, SW3 SW_Push, U1 XIAO-RP2040-DIP

Commit message: KiCad Fix
Connections:
- SW2 pad 2: unconnected-(SW2-Pad2) -> GND
- SW3 pad 1: /SW2 -> /SW3
Routing:
- net /SW3: track 0.84 -> 33.9 mm
- net GND: track 122.4 -> 125.3 mm, vias 3 -> 4
Changed lines of the file:
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@@
 	(net 8 "/LED3")
 	(net 9 "/SW1")
-	(net 10 "unconnected-(SW2-Pad2)")
-	(net 11 "/SW2")
-	(net 12 "unconnected-(U1-GPIO1{slash}RX-Pad8)")
-	(net 13 "unconnected-(U1-GPIO3{slash}MOSI-Pad11)")
-	(net 14 "unconnected-(U1-GPIO4{slash}MISO-Pad10)")
-	(net 15 "unconnected-(U1-GPIO0{slash}TX-Pad7)")
-	(net 16 "unconnected-(U1-3V3-Pad12)")
-	(net 17 "unconnected-(U1-GPIO2{slash}SCK-Pad9)")
-	(net 18 "/SW3")
+	(net 10 "/SW2")
+	(net 11 "unconnected-(U1-GPIO1{slash}RX-Pad8)")
+	(net 12 "unconnected-(U1-GPIO3{slash}MOSI-Pad11)")
+	(net 13 "unconnected-(U1-GPIO4{slash}MISO-Pad10)")
+	(net 14 "unconnected-(U1-GPIO0{slash}TX-Pad7)")
+	(net 15 "unconnected-(U1-3V3-Pad12)")
+	(net 16 "unconnected-(U1-GPIO2{slash}SCK-Pad9)")
+	(net 17 "/SW3")
 	(footprint "LED_THT:LED_D5.0mm"
 		(layer "F.Cu")
@@
 			(layers "F.Cu" "F.Mask")
 			(roundrect_rratio 0.1)
-			(net 11 "/SW2")
+			(net 10 "/SW2")
 			(pinfunction "GPIO27/ADC1/A1")
 			(pintype "passive")
@@
 			(layers "*.Cu" "*.Mask")
 			(remove_unused_layers no)
-			(net 11 "/SW2")
+			(net 10 "/SW2")
 			(pinfunction "GPIO27/ADC1/A1")
 			(pintype "passive")
@@
 			(layers "F.Cu" "F.Mask")
 			(roundrect_rratio 0.1)
-			(net 18 "/SW3")
+			(net 17 "/SW3")
 			(pinfunction "GPIO28/ADC2/A2")
 			(pintype "passive")
@@
 			(layers "*.Cu" "*.Mask")
 			(remove_unused_layers no)
-			(net 18 "/SW3")
+			(net 17 "/SW3")
 			(pinfunction "GPIO28/ADC2/A2")
 			(pintype "passive")
@@
 			(layers "F.Cu" "F.Mask")
 			(roundrect_rratio 0.1)
-			(net 15 "unconnected-(U1-GPIO0{slash}TX-Pad7)")
+			(net 14 "unconnected-(U1-GPIO0{slash}TX-Pad7)")
 			(pinfunction "GPIO0/TX")
 			(pintype "passive")
@@
 			(layers "*.Cu" "*.Mask")
 			(remove_unused_layers no)
-			(net 15 "unconnected-(U1-GPIO0{slash}TX-Pad7)")
+			(net 14 "unconnected-(U1-GPIO0{slash}TX-Pad7)")
 			(pinfunction "GPIO0/TX")
 			(pintype "passive")
@@
 			(layers "*.Cu" "*.Mask")
 			(remove_unused_layers no)
-			(net 12 "unconnected-(U1-GPIO1{slash}RX-Pad8)")
+			(net 11 "unconnected-(U1-GPIO1{slash}RX-Pad8)")
 			(pinfunction "GPIO1/RX")
 			(pintype "passive")
@@
 			(layers "F.Cu" "F.Mask")
 			(roundrect_rratio 0.1)
-			(net 12 "unconnected-(U1-GPIO1{slash}RX-Pad8)")
+			(net 11 "unconnected-(U1-GPIO1{slash}RX-Pad8)")
 			(pinfunction "GPIO1/RX")
 			(pintype "passive")
@@
 			(layers "*.Cu" "*.Mask")
 			(remove_unused_layers no)
-			(net 17 "unconnected-(U1-GPIO2{slash}SCK-Pad9)")
+			(net 16 "unconnected-(U1-GPIO2{slash}SCK-Pad9)")
 			(pinfunction "GPIO2/SCK")
 			(pintype "passive")
@@
 			(layers "F.Cu" "F.Mask")
 			(roundrect_rratio 0.1)
-			(net 17 "unconnected-(U1-GPIO2{slash}SCK-Pad9)")
+			(net 16 "unconnected-(U1-GPIO2{slash}SCK-Pad9)")
 			(pinfunction "GPIO2/SCK")
 			(pintype "passive")
@@
 			(layers "*.Cu" "*.Mask")
 			(remove_unused_layers no)
-			(net 14 "unconnected-(U1-GPIO4{slash}MISO-Pad10)")
+			(net 13 "unconnected-(U1-GPIO4{slash}MISO-Pad10)")
 			(pinfunction "GPIO4/MISO")
 			(pintype "passive")
@@
 			(layers "F.Cu" "F.Mask")
 			(roundrect_rratio 0.1)
-			(net 14 "unconnected-(U1-GPIO4{slash}MISO-Pad10)")
+			(net 13 "unconnected-(U1-GPIO4{slash}MISO-Pad10)")
 			(pinfunction "GPIO4/MISO")
 			(pintype "passive")
@@
 			(layers "*.Cu" "*.Mask")
 			(remove_unused_layers no)
-			(net 13 "unconnected-(U1-GPIO3{slash}MOSI-Pad11)")
+			(net 12 "unconnected-(U1-GPIO3{slash}MOSI-Pad11)")
 			(pinfunction "GPIO3/MOSI")
 			(pintype "passive")
@@
 			(layers "F.Cu" "F.Mask")
 			(roundrect_rratio 0.1)
-			(net 13 "unconnected-(U1-GPIO3{slash}MOSI-Pad11)")
+			(net 12 "unconnected-(U1-GPIO3{slash}MOSI-Pad11)")
 			(pinfunction "GPIO3/MOSI")
 			(pintype "passive")
@@
 			(layers "*.Cu" "*.Mask")
 			(remove_unused_layers no)
-			(net 16 "unconnected-(U1-3V3-Pad12)")
+			(net 15 "unconnected-(U1-3V3-Pad12)")
 			(pinfunction "3V3")
 			(pintype "passive")
@@
 			(layers "F.Cu" "F.Mask")
 			(roundrect_rratio 0.1)
-			(net 16 "unconnected-(U1-3V3-Pad12)")
+			(net 15 "unconnected-(U1-3V3-Pad12)")
 			(pinfunction "3V3")
 			(pintype "passive")
@@
 			(layers "*.Cu" "*.Mask")
 			(remove_unused_layers no)
-			(net 11 "/SW2")
+			(net 10 "/SW2")
 			(pinfunction "1")
 			(pintype "passive")
@@
 			(layers "*.Cu" "*.Mask")
 			(remove_unused_layers no)
-			(net 10 "unconnected-(SW2-Pad2)")
+			(net 2 "GND")
 			(pinfunction "2")
 			(pintype "passive")
@@
 			(layers "*.Cu" "*.Mask")
 			(remove_unused_layers no)
-			(net 11 "/SW2")
+			(net 17 "/SW3")
 			(pinfunction "1")
 			(pintype "passive")
@@
 	)
 	(segment
+		(start 110.38 105.3)
+		(end 109.601 104.521)
+		(width 0.2)
+		(layer "F.Cu")
+		(net 2)
+	)
+	(segment
 		(start 126.38 133.59)
 		(end 132.91 127.06)
@@
 	)
 	(segment
+		(start 110.38 107.135)
+		(end 110.38 105.3)
+		(width 0.2)
+		(layer "F.Cu")
+		(net 2)
+	)
+	(segment
 		(start 132.91 102.8817)
 		(end 132.91 112.16)
@@
 	)
 	(via
+		(at 109.601 104.521)
+		(size 0.6)
+		(drill 0.3)
+		(layers "F.Cu" "B.Cu")
+		(net 2)
+	)
+	(via
 		(at 140.5 81.97)
 		(size 0.6)
@@
 		(width 0.2)
 		(layer "F.Cu")
-		(net 11)
+		(net 10)
 	)
 	(segment
@@
 		(width 0.2)
 		(layer "F.Cu")
-		(net 11)
+		(net 10)
 	)
 	(segment
@@
 		(width 0.2)
 		(layer "F.Cu")
-		(net 11)
+		(net 10)
 	)
 	(segment
@@
 		(width 0.2)
 		(layer "F.Cu")
-		(net 11)
+		(net 10)
 	)
 	(segment
@@
 		(width 0.2)
 		(layer "B.Cu")
-		(net 11)
+		(net 10)
 	)
 	(segment
@@
 		(width 0.2)
 		(layer "B.Cu")
-		(net 11)
+		(net 10)
 	)
 	(segment
@@
 		(width 0.2)
 		(layer "B.Cu")
-		(net 11)
+		(net 10)
 	)
 	(segment
@@
 		(width 0.2)
 		(layer "B.Cu")
-		(net 11)
+		(net 10)
 	)
 	(segment
@@
 		(width 0.2)
 		(layer "B.Cu")
-		(net 11)
+		(net 10)
 	)
 	(segment
@@
 		(width 0.2)
 		(layer "F.Cu")
-		(net 12)
+		(net 11)
 	)
 	(segment
@@
 		(width 0.2)
 		(layer "F.Cu")
-		(net 13)
+		(net 12)
 	)
 	(segment
@@
 		(width 0.2)
 		(layer "F.Cu")
-		(net 14)
+		(net 13)
 	)
 	(segment
@@
 		(width 0.2)
 		(layer "F.Cu")
-		(net 15)
+		(net 14)
 	)
 	(segment
@@
 		(width 0.2)
 		(layer "F.Cu")
-		(net 16)
+		(net 15)
 	)
 	(segment
@@
 		(width 0.2)
 		(layer "F.Cu")
+		(net 16)
+	)
+	(segment
+		(start 141.62 131.05)
+		(end 138.017 134.653)
+		(width 0.2)
+		(layer "F.Cu")
+		(net 17)
+	)
+	(segment
+		(start 138.017 134.653)
+		(end 123.49953 134.653)
+		(width 0.2)
+		(layer "F.Cu")
+		(net 17)
+	)
+	(segment
+		(start 123.49953 134.653)
+		(end 116.73 127.88347)
+		(width 0.2)
+		(layer "F.Cu")
 		(net 17)
 	)
@@
 		(width 0.2)
 		(layer "F.Cu")
-		(net 18)
+		(net 17)
+	)
+	(segment
+		(start 116.73 127.88347)
+		(end 116.73 124.046)
+		(width 0.2)
+		(layer "F.Cu")
+		(net 17)
 	)
 	(zone
